File: HARDWARE/eduArdu_Rev_B/eduArdu_Rev_B.kicad_pcb (KiCad board)
At the start: 2 copper layers, 170.2 x 70.9 mm, 117 parts, among them Q1 16.000MHz/SMD5x3.2/12pF, SW1 T1107A(6x3,8x2,5MM), U1 BL4054B-42TPRN(SOT23-5), U10 LM358, U2 ATmega32U4-AU, U3 RPM7236-H8, U4 TCN75, U5 74HC595, U6 74HC595, U7 ULN2003AD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

Commit message: label D13 changed to D23
Other:
- board text added: "D23"
- board text removed: "D13"
Changed lines of the file:
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@@
     (effects (font (size 1.5 1.5) (thickness 0.3)))
   )
-  (gr_text D13 (at 99 71.5) (layer F.SilkS)
+  (gr_text D23 (at 99 71.5) (layer F.SilkS)
     (effects (font (size 1.5 1.5) (thickness 0.3)))
   )
